File: uav/landing-gear/pcb/pcb.kicad_pcb (KiCad board)
At the start: 2 copper layers, 21.8 x 14.2 mm, 17 parts, among them J1 LimitSW1, J2 ICSP, J3 LimitSW2, J4 Motor, J5 ULink, U1 PIC16F15223-I/MG, U2 TLV75733PDBV, U3 DRV8837

Commit message: r
Parts:
- U3: footprint Package_SON:WSON-8-1EP_2x2mm_P0.5mm_EP0.9x1.6mm -> Package_SON:WSON-8-1EP_2x2mm_P0.5mm_EP0.9x1.6mm_ThermalVias
Routing:
- net GNDREF: vias 17 -> 14
Other:
- board text added: "V1"
Changed lines of the file:
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@@
 		)
 	)
-	(footprint "Package_SON:WSON-8-1EP_2x2mm_P0.5mm_EP0.9x1.6mm"
+	(footprint "Package_SON:WSON-8-1EP_2x2mm_P0.5mm_EP0.9x1.6mm_ThermalVias"
 		(layer "F.Cu")
 		(at 156.8 101.8 90)
 		(descr "8-Lead Plastic WSON, 2x2mm Body, 0.5mm Pitch, WSON-8, http://www.ti.com/lit/ds/symlink/lm27761.pdf")
-		(tags "WSON 8 1EP")
+		(tags "WSON 8 1EP ThermalVias")
 		(property "Reference" "U3"
-			(at -1.2 1.65 90)
+			(at -1.1 1.675 90)
 			(layer "F.SilkS")
 			(effects
 				(font
 					(size 0.5 0.5)
-					(thickness 0.15)
+					(thickness 0.125)
 				)
 			)
@@
 			)
 		)
-		(property "Datasheet" "http://www.ti.com/lit/ds/symlink/drv8837.pdf"
+		(property "Datasheet" "https://www.ti.com/lit/ds/symlink/drv8212p.pdf"
 			(at 0 0 90)
 			(unlocked yes)
@@
 			)
 		)
-		(property "Description" "H-Bridge driver, 1.8A, Low Voltage, PWM input, WSON-8"
+		(property "Description" "H-Bridge driver, 4A, Low Voltage, PWM input, WSON-8"
 			(at 0 0 90)
 			(unlocked yes)
@@
 			(pintype "power_in")
 		)
+		(pad "9" thru_hole circle
+			(at 0 -0.5 90)
+			(size 0.6 0.6)
+			(drill 0.25)
+			(property pad_prop_heatsink)
+			(layers "*.Cu")
+			(remove_unused_layers no)
+			(net 3 "GNDREF")
+			(pinfunction "GND")
+			(pintype "passive")
+		)
 		(pad "9" smd rect
 			(at 0 0 90)
 			(size 0.9 1.6)
 			(layers "F.Cu" "F.Mask")
+			(net 3 "GNDREF")
+			(pinfunction "GND")
+			(pintype "passive")
+		)
+		(pad "9" smd rect
+			(at 0 0 90)
+			(size 0.9 1.6)
+			(layers "B.Cu")
+			(net 3 "GNDREF")
+			(pinfunction "GND")
+			(pintype "passive")
+		)
+		(pad "9" thru_hole circle
+			(at 0 0.5 90)
+			(size 0.6 0.6)
+			(drill 0.25)
+			(property pad_prop_heatsink)
+			(layers "*.Cu")
+			(remove_unused_layers no)
 			(net 3 "GNDREF")
 			(pinfunction "GND")
@@
 		)
 	)
+	(gr_text "V1"
+		(at 165.4 102.15 0)
+		(layer "F.SilkS")
+		(effects
+			(font
+				(size 1.5 1.5)
+				(thickness 0.3)
+				(bold yes)
+			)
+		)
+	)
 	(gr_text "CLK"
 		(at 164.7 98.1 0)
@@
 	)
 	(via
-		(at 157.3 101.8)
-		(size 0.459)
-		(drill 0.255)
-		(layers "F.Cu" "B.Cu")
-		(net 3)
-	)
-	(via
 		(at 154.85 101.11)
 		(size 0.459)
@@
 	)
 	(via
-		(at 156.3 101.8)
-		(size 0.459)
-		(drill 0.255)
-		(layers "F.Cu" "B.Cu")
-		(net 3)
-	)
-	(via
 		(at 152.79 103.9)
 		(size 0.459)
@@
 		(size 0.459)
 		(drill 0.255)
-		(layers "F.Cu" "B.Cu")
-		(net 3)
-	)
-	(via
-		(at 156.8 101.8)
-		(size 0.459)
-		(drill 0.255)

Commit message: clean drc
Parts:
- removed J2: ICSP, Connector_PinHeader_1.27mm:PinHeader_1x04_P1.27mm_Vertical
- C4: value 10n -> 100n
- J5: footprint Connector_JST:JST_ZH_B4B-ZR_1x04_P1.50mm_Vertical -> Connector_JST:JST_ZH_B5B-ZR_1x05_P1.50mm_Vertical
- moved J3 18.2 mm to (165.1, 97.3), turned to 90 degrees
- moved C4 2.93 mm to (163.1, 101.4), turned to 90 degrees
- moved J5 1.50 mm to (148.0, 97.1)
- moved J4 0.85 mm to (155.7, 105.5)
- moved C2 0.69 mm to (152.6, 103.9)
- moved R3 0.07 mm to (161.0, 100.4)
Connections:
- C1 pad 2: GNDREF -> GND
- C2 pad 2: GNDREF -> GND
- C3 pad 1: GNDREF -> GND
- C4 pad 2: GNDREF -> GND
- C5 pad 1: GNDREF -> GND
- C6 pad 2: GNDREF -> GND
- J1 pad 2: GNDREF -> GND
- J3 pad 1: RA2 -> GND
- J3 pad 2: GNDREF -> RA2
- J5 pad 1: GNDREF -> GND
- J5 pad 2: SCL -> SDA
- J5 pad 3: SDA -> SCL
- U1 pad 11: Net-(J2-Pin_2) -> SCL
- U1 pad 12: Net-(J2-Pin_3) -> SDA
- U1 pad 13: GNDREF -> GND
- U1 pad 17: GNDREF -> GND
- U1 pad 8: SDA -> unconnected-(U1-RC1-Pad8)
- U1 pad 9: SCL -> unconnected-(U1-RC0-Pad9)
- U2 pad 2: GNDREF -> GND
- U3 pad 4: GNDREF -> GND
- U3 pad 9: GNDREF -> GND
Routing:
- net RA2: track 36.5 -> 8.66 mm
- net MCLR: track 9.27 -> 23.5 mm, vias 1 -> 0
- net Net-(J2-Pin_3): track 12.2 -> 0.00 mm
- net Net-(J2-Pin_2): track 11.3 -> 0.00 mm
- net SCL: track 10.4 -> 17.6 mm, vias 1 -> 0
- net GND: track 0.00 -> 6.00 mm, vias 0 -> 16
- net GNDREF: track 5.55 -> 0.00 mm, vias 14 -> 0
- net VDC: track 7.44 -> 12.2 mm, vias 6 -> 7
- net SDA: track 11.1 -> 10.8 mm, vias 1 -> 0
- added copper zone on B.Cu, net GND
- added copper zone on F.Cu, net GND
- removed copper zone on B.Cu, net GNDREF
- removed copper zone on F.Cu, net GNDREF
Other:
- board size 21.8 x 14.2 mm -> 22.5 x 14.2 mm
- board text added: "PRGM"
- board text added: "SCL"
- board text added: "SDA"
- board text added: "V2"
- board text added: "VDC"
- board text removed: "CLK"
- board text removed: "DAT"
- board text removed: "V1"
